File: diseño/diseño.kicad_pcb (KiCad board)
At the start: 2 copper layers, 96 x 94 mm, 21 parts

Commit message: Trabajo completo
Routing:
- net Net-(Bootstrap1-Pin_2): track 0.00 -> 242.0 mm
- net Net-(DRL1-A): track 0.00 -> 158.1 mm
- net Net-(DRU1-K): track 0.00 -> 105.1 mm, vias 0 -> 1
- net Net-(SU1-C): track 0.00 -> 94.9 mm
- net Net-(TS1-Pin_1): track 0.00 -> 92.8 mm
- net Net-(Dv1-K): track 0.00 -> 83.1 mm
- net Net-(DRL1-K): track 0.00 -> 57.6 mm
- net Net-(Dsl1-A): track 0.00 -> 44.5 mm
- net Net-(Dsu1-A): track 0.00 -> 37.2 mm
- net Net-(Bootstrap1-Pin_3): track 0.00 -> 24.2 mm
- net Net-(Bootstrap1-Pin_1): track 0.00 -> 15.5 mm
